File: bank6_7.kicad_sch (KiCad schematic)
At the start: 1 part, among them IC1 ECP5-BGA256

Commit message: sch: capture 16-bit bus
Connections:
- net GND: no longer IC1.G2 (PL14B), IC1.G3 (PL14C), IC1.H2 (PL20B), IC1.H3 (PL14D)
- net VCCRAM: no longer IC1.J1 (PL23A), IC1.J2 (PL23B), IC1.J3 (PL20C)
- net RAM.DQ8: now reaches IC1.F1 (PL14A)
- net RAM.DM1: now reaches IC1.G1 (PL20A)
- net RAM.RWDS renamed RAM.DM0
- net RAM.~{CK}: no longer names the net of IC1.D3 (PL2D)
- net RAM.~{RESET}: no longer names the net of IC1.C1 (PL5A)
- new net RAM.DQ10: IC1.G3 (PL14C)
- new net RAM.DQ11: IC1.H3 (PL14D)
- new net RAM.DQ12: IC1.J3 (PL20C)
- new net RAM.DQ13: IC1.H2 (PL20B)
- new net RAM.DQ14: IC1.J1 (PL23A)
- new net RAM.DQ15: IC1.J2 (PL23B)
- new net RAM.DQ9: IC1.G2 (PL14B)

Commit message: routing is possible?
Connections:
- net RAM.DM0: now also IC1.G1 (PL20A); no longer IC1.D1 (PL8A)
- net RAM.DM1: now also IC1.B1 (PL2A); no longer IC1.G1 (PL20A)
- net RAM.DQ0: now also IC1.J2 (PL23B); no longer IC1.F2 (PL11C)
- net RAM.DQ1: now also IC1.G3 (PL14C); no longer IC1.B1 (PL2A)
- net RAM.DQ10: now also IC1.D1 (PL8A); no longer IC1.G3 (PL14C)
- net RAM.DQ11: now also IC1.F3 (PL5D); no longer IC1.H3 (PL14D)
- net RAM.DQ12: now also IC1.E3 (PL5C); no longer IC1.J3 (PL20C)
- net RAM.DQ13: now also IC1.E2 (PL8B); no longer IC1.H2 (PL20B)
- net RAM.DQ14: now also IC1.C2 (PL5B); no longer IC1.J1 (PL23A)
- net RAM.DQ15: now also IC1.E1 (PL11D); no longer IC1.J2 (PL23B)
- net RAM.DQ2: now also IC1.G2 (PL14B); no longer IC1.C2 (PL5B)
- net RAM.DQ3: now also IC1.H2 (PL20B); no longer IC1.E1 (PL11D)
- net RAM.DQ4: now also IC1.F1 (PL14A); no longer IC1.E3 (PL5C)
- net RAM.DQ5: now also IC1.H3 (PL14D); no longer IC1.E2 (PL8B)
- net RAM.DQ6: now also IC1.J1 (PL23A); no longer IC1.F3 (PL5D)
- net RAM.DQ7: now also IC1.J3 (PL20C); no longer IC1.G4 (PL11B)
- net RAM.DQ8: now also IC1.F2 (PL11C); no longer IC1.F1 (PL14A)
- net RAM.DQ9: now also IC1.G4 (PL11B); no longer IC1.G2 (PL14B)
