File: bank6_7.kicad_sch (KiCad schematic)
At the start: 1 part, among them IC1 ECP5-BGA256

Commit message: length match all dqs/dq to +/- 2mm
Connections:
- net RAM.DQ10: now also IC1.F2 (PL11C); no longer IC1.D1 (PL8A)
- net RAM.DQ11: now also IC1.G4 (PL11B); no longer IC1.F3 (PL5D)
- net RAM.DQ6: now also IC1.J3 (PL20C); no longer IC1.J1 (PL23A)
- net RAM.DQ7: now also IC1.J1 (PL23A); no longer IC1.J3 (PL20C)
- net RAM.DQ8: now also IC1.F3 (PL5D); no longer IC1.F2 (PL11C)
- net RAM.DQ9: now also IC1.D1 (PL8A); no longer IC1.G4 (PL11B)
Changed lines of the file:
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@@
 	)
 	(label "RAM.DQ10"
-		(at 204.47 77.47 0)
+		(at 204.47 93.98 0)
 		(effects
 			(font
@@
 	)
 	(label "RAM.DQ11"
-		(at 204.47 72.39 0)
+		(at 204.47 91.44 0)
 		(effects
 			(font
@@
 	)
 	(label "RAM.DQ6"
-		(at 203.2 137.16 0)
+		(at 203.2 129.54 0)
 		(effects
 			(font
@@
 	)
 	(label "RAM.DQ8"
-		(at 204.47 93.98 0)
+		(at 204.47 72.39 0)
 		(effects
 			(font
@@
 	)
 	(label "RAM.DQ7"
-		(at 203.2 129.54 0)
+		(at 203.2 137.16 0)
 		(effects
 			(font
@@
 	)
 	(label "RAM.DQ9"
-		(at 204.47 91.44 0)
-		(effects
-			(font
+		(at 204.47 77.47 0)
+		(effects
+			(font

Commit message: swap dq9/dm1 after pnr route test
Connections:
- net RAM.DM1: now also IC1.D1 (PL8A); no longer IC1.B1 (PL2A)
- net RAM.DQ9: now also IC1.B1 (PL2A); no longer IC1.D1 (PL8A)
Changed lines of the file:
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@@
 	)
 	(label "RAM.DM1"
-		(at 204.47 52.07 0)
+		(at 204.47 77.47 0)
 		(effects
 			(font
@@
 	)
 	(label "RAM.DQ9"
-		(at 204.47 77.47 0)
+		(at 204.47 52.07 0)
 		(effects
 			(font
